Commit message: up to date

File: src/f112th_sim_2024_alpha/description/gazebo_control.xacro (robot description, xacro)
@@ -13,8 +13,9 @@
             <max_wheel_acceleration>10.0</max_wheel_acceleration>
             <!-- outputs -->
-            <odometry_frame>odom</odometry_frame>
+            <odometry_frame>odom_sim</odometry_frame>
+            <odometryTopic>odom_sim</odometryTopic>
             <robot_base_frame>base_link</robot_base_frame>
-            <publish_odom>true</publish_odom>
-            <publish_odom_tf>true</publish_odom_tf>
+            <publish_odom>false</publish_odom>
+            <publish_odom_tf>false</publish_odom_tf>
             <publish_wheel_tf>true</publish_wheel_tf>
         </plugin>

File: src/f112th_sim_2024_alpha/description/imu.urdf.xacro (robot description, xacro)
@@ -50,5 +50,5 @@
                 <ros>
                     <!--Output topic: scan-->
-                    <remapping>~/out:=imu</remapping>
+                    <remapping>~/out:=/alpha/imu</remapping>
                 </ros>
             </plugin>

File: src/f112th_sim_2024_alpha/description/lidar.xacro (robot description, xacro)
@@ -49,5 +49,5 @@
             <plugin name="laser_controller" filename="libgazebo_ros_ray_sensor.so">
                 <ros>
-                    <remapping>~/out:=scan</remapping>
+                    <remapping>~/out:=/alpha/scan</remapping>
                 </ros>
                 <output_type>sensor_msgs/LaserScan</output_type>

File: src/f112th_sim_2024_alpha/description/robot_core.xacro (robot description, xacro)
@@ -17,4 +17,12 @@
     <!-- Example link -->
     <xacro:include filename="inertial_macros.xacro"/>
+    <joint name="base_footprint_joint" type="fixed">
+        <parent link="base_link"/>
+        <child link="base_footprint"/>
+        <origin xyz="0 0 0"/>
+    </joint>
+    <!-- Example link -->
+    <link name="base_footprint">
+    </link>
     <!-- Example link -->
     <link name="base_link">

Commit message: Entrega Final

File: src/f112th_sim_2024_alpha/description/gazebo_control.xacro (robot description, xacro)
@@ -7,5 +7,5 @@
             <left_joint>left_wheel_joint</left_joint>
             <right_joint>right_wheel_joint</right_joint>
-            <wheel_separation>0.35</wheel_separation>
+            <wheel_separation>0.25</wheel_separation>
             <wheel_diameter>0.1</wheel_diameter>
             <!-- limits -->
@@ -13,6 +13,6 @@
             <max_wheel_acceleration>10.0</max_wheel_acceleration>
             <!-- outputs -->
-            <odometry_frame>odom_sim</odometry_frame>
-            <odometryTopic>odom_sim</odometryTopic>
+            <odometry_frame>odom</odometry_frame>
+            <odometryTopic>odom</odometryTopic>
             <robot_base_frame>base_link</robot_base_frame>
             <publish_odom>true</publish_odom>

File: src/f112th_sim_2024_alpha/description/lidar.xacro (robot description, xacro)
@@ -42,5 +42,5 @@
                 </scan>
                 <range>
-                    <min>0.3</min>
+                    <min>0.1</min>
                     <max>12</max>
                     <resolution>0.01</resolution>

File: src/f112th_sim_2024_alpha/description/odom_tf_robot/lidar.xacro (robot description, xacro)
@@ -13,5 +13,4 @@
                 <cylinder radius="0.035" length="0.02"/>
             </geometry>
-            <material name="red"/>
         </visual>
         <collision>

File: src/f112th_sim_2024_alpha/description/odom_tf_robot/odom_to_tf.urdf.xacro (robot description, xacro)
@@ -45,5 +45,4 @@
                 <cylinder radius="0.035" length="0.02"/>
             </geometry>
-            <material name="red"/>
         </visual>
         <collision>

File: src/f112th_sim_2024_alpha/description/robot_core.xacro (robot description, xacro)
@@ -38,5 +38,5 @@
             <origin xyz="0.15 0 0.075"/>
             <geometry>
-                <box size="0.3 0.3 0.15"/>
+                <box size="0.3 0.18 0.15"/>
             </geometry>
             <material name="white"/>
@@ -45,5 +45,5 @@
             <origin xyz="0.15 0 0.075"/>
             <geometry>
-                <box size="0.3 0.3 0.15"/>
+                <box size="0.3 0.18 0.15"/>
             </geometry>
         </collision>
@@ -56,5 +56,5 @@
         <parent link="base_link"/>
         <child link="left_wheel"/>
-        <origin xyz="0 0.175 0" rpy="-${pi/2} 0 0"/>
+        <origin xyz="0 0.111 0" rpy="-${pi/2} 0 0"/>
         <axis xyz="0 0 1"/>
     </joint>
@@ -85,5 +85,5 @@
         <parent link="base_link"/>
         <child link="right_wheel"/>
-        <origin xyz="0 -0.175 0" rpy="${pi/2} 0 0"/>
+        <origin xyz="0 -0.111 0" rpy="${pi/2} 0 0"/>
         <axis xyz="0 0 -1"/>
     </joint>
